File: hardware/WeighFi.sch (KiCad schematic (older format))
At the start: 51 parts, among them P1 CONN_1, P2 CONN_1, P3 CONN_1, U1 MAX1555, U2 MCP1700

Commit message: Add power switch, rearrange layout on page
Parts:
- added C?: 10nF, symbol C
- added R? (x2): R, symbol R
- added S?: SWITCH_DP4T, symbol SWITCH_DP4T
Connections:
- net +3V: now also C4.1, S?.4, S?.5, S?.6; no longer U2.VO
- net +BATT: now also R?.1, S?.1; no longer C4.1, U2.VI
- net ADC_CLOCK: now also U?.26 ((T1/OC4D/ADC9)_PD6)
- net ADC_DATA: now also U?.27 ((T0/OC4D/ADC10)_PD7)
- net ADC_PWRDN: now also U?.22 ((XCK1/CTS)_PD5)
- net ADC_SPEED: now also U?.25 ((PCINT20/XCK/T0)_PD4)
- net GND: now also C?.2, R?.2, S?.2
- net SW_ST: now reaches U?.12 ((PCINT7/OC0A/OC1C/RTS)_PB7)
- net SW_ST: now also S?.10
- net SW_KG: now reaches U?.29 ((PCINT5/OC1A/OC4B/ADC12)_PB5)
- net SW_KG: now also S?.8
- net SW_LB: now reaches U?.30 ((PCINT6/OC1B/OC4B/ADC13)_PB6)
- net SW_LB: now also S?.9
- net BAT_ADC: now reaches U?.41 ((ADC0)_PF0)
- net BAT_ADC: now also C?.1, R?.1, R?.2
- no-connect marks 19 -> 21
Other:
- note added: "Normally SJ2 would be connected to ground for \ninternal clock. If clock speed needs to be overriden \nby MCU then connect SJ1 instead. Note that \nLCD_CLOCK *must* be supplied by MCU in this case"
- note added: "Optional circuitry to support\nwake on CTS or received data"
- moved on the sheet: C4, C5, C?, H1, H2, H3, H4, ISP1, P3, P?, Q?, R?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

Commit message: Hook up more connections, re-arrange the page again
Parts:
- added P?: CONN_4, symbol CONN_4
Connections:
- net +3V: now also U2.VO; no longer C4.1, S?.4, S?.5, S?.6
- net +BATT: now also P?.3
- net ADC_PWRDN: now also U?.32 ((ICP3/CLK0/OC4A)_PC7); no longer U?.22 ((XCK1/CTS)_PD5)
- net ADC_SPEED: now also U?.31 ((OC3A/OC4A)_PC6); no longer U?.25 ((PCINT20/XCK/T0)_PD4)
- net E-: now also P?.4
- net I2C_CLOCK: now also U?.18 ((OC0B/SCL/INT0)_PD0); no longer U?.20 ((RXD1/INT2)_PD2)
- net S+: now also P?.1
- net S-: now also P?.2
- net SW_KG: now also U?.28 ((PCINT4/ADC11)_PB4); no longer U?.29 ((PCINT5/OC1A/OC4B/ADC12)_PB5)
- net SW_LB: now also U?.29 ((PCINT5/OC1A/OC4B/ADC12)_PB5); no longer U?.30 ((PCINT6/OC1B/OC4B/ADC13)_PB6)
- net SW_ST: now also U?.30 ((PCINT6/OC1B/OC4B/ADC13)_PB6); no longer U?.12 ((PCINT7/OC0A/OC1C/RTS)_PB7)
- net WIFI_ASSOC: now also U?.38 ((TMS/ADC5)_PF5)
- net WIFI_CTS: now also U?.12 ((PCINT7/OC0A/OC1C/RTS)_PB7)
- net WIFI_RTS: now also U?.22 ((XCK1/CTS)_PD5)
- net WIFI_RX: now also U?.21 ((TXD1/INT3)_PD3)
- net WIFI_SLEEP: now also U?.37 ((TDO/ADC6)_PF6)
- net WIFI_TX: now also U?.20 ((RXD1/INT2)_PD2)
- net PWR_SW_OUT: now reaches U2.VI
- net PWR_SW_OUT: now also C4.1, S?.4, S?.5, S?.6
- net WIFI_RESET: now reaches MOD?.40 (RESET)
- net WIFI_WAKE: now reaches MOD?.41 (FORCE_AWAKE)
- net WIFI_WAKE: now also U?.36 ((TDI/ADC7)_PF7)
Other:
- note added: "External ADC"
- note added: "In System Programming header"
- note added: "LCD Driver"
- note added: "MCU"
- note added: "Main power and unit selection switch"
- note added: "Power control for LCD driver"
- note added: "Strain gauge connector"
- note added: "The RTS and CTS signals are unlikely to be used,\ncould be dropped if routing is problematic."
- note added: "Voltage divider for \nbattery measurements \nusing internal ADC"
- note added: "WiFi Module"
- note removed: "ADC"
- note removed: "In System Programming"
- moved on the sheet: BT1, C1, C2, C3, C4, C5, H1, H2, H3, H4, ISP1, P1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

Commit message: Initial schematic annotation and ERC checking
Parts:
- gave numbers to parts that had none: 40
- renumbered C4 to C12, C5 to C15
Connections:
- net LCD_ENABLE: now also U3.25 ((PCINT20/XCK/T0)_PD4)
- no-connect marks 21 -> 36
Other:
- note added: "Power control for LCD driver\n(reduce sleep current)"
- note removed: "Power control for LCD driver"

Commit message: Start adding test points to signal lines, connect LCD driver clock input to MCU output compare pin
Parts:
- added P1, P11, P12, P13, P14, P15, P16, P17, P18, P2, P3, P4, P7, P9: CONN_1, symbol CONN_1
- renumbered P4 to P10, P5 to P19, P1 to P5, P2 to P6, P3 to P8
Connections:
- net +BATT: now also P15.1
- net ADC_CLOCK: now also P16.1
- net ADC_DATA: now also P18.1
- net ADC_PWRDN: now also P14.1
- net ADC_SPEED: now also P12.1
- net BAT_ADC: now also P4.1
- net E-: now also P17.1
- net LCD_CLOCK: now also U3.29 ((PCINT5/OC1A/OC4B/ADC12)_PB5)
- net LCD_ENABLE: now also P7.1
- net LCD_SUPPLY: now also P9.1
- net S+: now also P11.1
- net S-: now also P13.1
- net SW_KG: now also U3.30 ((PCINT6/OC1B/OC4B/ADC13)_PB6), P1.1; no longer U3.28 ((PCINT4/ADC11)_PB4)
- net SW_LB: now also U3.28 ((PCINT4/ADC11)_PB4), P2.1; no longer U3.29 ((PCINT5/OC1A/OC4B/ADC12)_PB5)
- net SW_ST: now also U3.8 ((PCINT0/SS)_PB0), P3.1; no longer U3.30 ((PCINT6/OC1B/OC4B/ADC13)_PB6)

Commit message: Add charging status indicator, connect WiFi module reset line to MCU
Parts:
- added D1: LED, symbol LED
- added R12: 1K8, symbol R
- renumbered R12 to R13, R13 to R14
Connections:
- net CHG: now also R12.1
- net GND: now also D1.2 (K)
- net WIFI_RESET: now also U3.39 ((TCK/ADC4)_PF4)
- new net: D1.1 (A), R12.2
Other:
- note added: "Charging status display"

Commit message: Add switch to reset line for bootloader entry, tie HWB to ground
Parts:
- added S2: SWITCH_SPST, symbol SWITCH_SPST
Connections:
- net GND: now also U3.33 ((HWB)_PE2), S2.1
- net RST: now also S2.2

Commit message: Complete initial ERC
Connections:
- no-connect marks 36 -> 38
Changed lines of the file:
@@
-EESchema Schematic File Version 2  date Mon 04 Jun 2012 18:57:13 BST
+EESchema Schematic File Version 2  date Mon 04 Jun 2012 19:01:00 BST
 LIBS:dresco
 LIBS:power
@@
 Comment4 ""
 $EndDescr
+$Comp
+L ATMEGA16U4/32U4 U3
+U 1 1 4FCCF7C0
+P 8700 5650
+F 0 "U3" H 8650 5750 50  0000 L BNN
+F 1 "ATMEGA16U4/32U4" H 8300 5920 50  0000 L BNN
+	1    8700 5650
+	1    0    0    -1
+$EndComp
+NoConn ~ 9800 4350
+NoConn ~ 9800 4950
 Wire Wire Line
 	10150 5100 10150 5050
@@
 	6000 3800 6000 4000
 $Comp
-L GND #PWR22
+L GND #PWR01
 U 1 1 4FCCF6AD
 P 10150 5100
-F 0 "#PWR22" H 10150 5100 30  0001 C CNN
+F 0 "#PWR01" H 10150 5100 30  0001 C CNN
 F 1 "GND" H 10150 5030 30  0001 C CNN
 	1    10150 5100
@@
 $EndComp
 $Comp
-L GND #PWR16
+L GND #PWR02
 U 1 1 4FCCF5F7
 P 6000 4000
-F 0 "#PWR16" H 6000 4000 30  0001 C CNN
+F 0 "#PWR02" H 6000 4000 30  0001 C CNN
 F 1 "GND" H 6000 3930 30  0001 C CNN
 	1    6000 4000
@@
 CHG
 $Comp
-L GND #PWR21
+L GND #PWR03
 U 1 1 4FCCE26F
 P 10050 2450
-F 0 "#PWR21" H 10050 2450 30  0001 C CNN
+F 0 "#PWR03" H 10050 2450 30  0001 C CNN
 F 1 "GND" H 10050 2380 30  0001 C CNN
 	1    10050 2450
@@
 NoConn ~ 3600 4950
 $Comp
-L PWR_FLAG #FLG3
+L PWR_FLAG #FLG04
 U 1 1 4FC509BC
 P 7150 2300
-F 0 "#FLG3" H 7150 2570 30  0001 C CNN
+F 0 "#FLG04" H 7150 2570 30  0001 C CNN
 F 1 "PWR_FLAG" H 7150 2530 30  0000 C CNN
 	1    7150 2300
@@
 $EndComp
 $Comp
-L PWR_FLAG #FLG4
+L PWR_FLAG #FLG05
 U 1 1 4FC50659
 P 8950 10000
-F 0 "#FLG4" H 8950 10095 30  0001 C CNN
+F 0 "#FLG05" H 8950 10095 30  0001 C CNN
 F 1 "PWR_FLAG" H 8950 10180 30  0000 C CNN
 	1    8950 10000
@@
 LCD_ENABLE
 $Comp
-L PWR_FLAG #FLG2
+L PWR_FLAG #FLG06
 U 1 1 4FC50360
 P 7150 1500
-F 0 "#FLG2" H 7150 1770 30  0001 C CNN
+F 0 "#FLG06" H 7150 1770 30  0001 C CNN
 F 1 "PWR_FLAG" H 7150 1730 30  0000 C CNN
 	1    7150 1500
@@
 NoConn ~ 2850 9700
 $Comp
-L GND #PWR3
+L GND #PWR07
 U 1 1 4FC34993
 P 1650 10400
-F 0 "#PWR3" H 1650 10400 30  0001 C CNN
+F 0 "#PWR07" H 1650 10400 30  0001 C CNN
 F 1 "GND" H 1650 10330 30  0001 C CNN
 	1    1650 10400
@@
 BAT_ADC
 $Comp
-L GND #PWR9
+L GND #PWR08
 U 1 1 4FBF8CF7
 P 5550 10400
-F 0 "#PWR9" H 5550 10400 30  0001 C CNN
+F 0 "#PWR08" H 5550 10400 30  0001 C CNN
 F 1 "GND" H 5550 10330 30  0001 C CNN
 	1    5550 10400
@@
 $EndComp
 $Comp
-L +BATT #PWR8
+L +BATT #PWR09
 U 1 1 4FBF8CD4
 P 5550 8900
-F 0 "#PWR8" H 5550 8850 20  0001 C CNN
+F 0 "#PWR09" H 5550 8850 20  0001 C CNN
 F 1 "+BATT" H 5550 9000 30  0000 C CNN
 	1    5550 8900
@@
 $EndComp
 $Comp
-L +VUSB #PWR12
+L +VUSB #PWR010
 U 1 1 4FBF89B4
 P 5900 5600
-F 0 "#PWR12" H 5900 5550 20  0001 C CNN
+F 0 "#PWR010" H 5900 5550 20  0001 C CNN
 F 1 "+VUSB" H 5900 5700 30  0000 C CNN
 	1    5900 5600
@@
 $EndComp
 $Comp
-L GND #PWR27
+L GND #PWR011
 U 1 1 4FBEC67F
 P 12150 4500
-F 0 "#PWR27" H 12150 4500 30  0001 C CNN
+F 0 "#PWR011" H 12150 4500 30  0001 C CNN
 F 1 "GND" H 12150 4430 30  0001 C CNN
 	1    12150 4500
@@
 LCD_ENABLE
 $Comp
-L +3V #PWR19
+L +3V #PWR012
 U 1 1 4FBEC3B3
 P 8450 9050
-F 0 "#PWR19" H 8450 8960 30  0001 C CNN
+F 0 "#PWR012" H 8450 8960 30  0001 C CNN
 F 1 "+3V" H 8450 9160 30  0000 C CNN
 	1    8450 9050
@@
 MOSI
 $Comp
-L GND #PWR13
+L GND #PWR013
 U 1 1 4FBE97EF
 P 5900 6300
-F 0 "#PWR13" H 5900 6300 30  0001 C CNN
+F 0 "#PWR013" H 5900 6300 30  0001 C CNN
 F 1 "GND" H 5900 6230 30  0001 C CNN
 	1    5900 6300
@@
 $EndComp
 $Comp
-L ATMEGA16U4/32U4 U3
-U 1 1 4FBE8375
-P 8700 5650
-F 0 "U3" H 8650 5750 50  0000 L BNN
-F 1 "ATMEGA16U4/32U4" H 8300 5920 50  0000 L BNN
-	1    8700 5650
-	1    0    0    -1
-$EndComp
-$Comp
 L C C7
 U 1 1 4FBE82BB
@@
 $EndComp
 $Comp
-L GND #PWR15
+L GND #PWR014
 U 1 1 4FBE8254
 P 5900 7350
-F 0 "#PWR15" H 5900 7350 30  0001 C CNN
+F 0 "#PWR014" H 5900 7350 30  0001 C CNN
 F 1 "GND" H 5900 7280 30  0001 C CNN
 	1    5900 7350
@@
 $EndComp
 $Comp
-L +3V #PWR14
+L +3V #PWR015
 U 1 1 4FBE823E
 P 5900 6550
-F 0 "#PWR14" H 5900 6460 30  0001 C CNN
+F 0 "#PWR015" H 5900 6460 30  0001 C CNN
 F 1 "+3V" H 5900 6660 30  0000 C CNN
 	1    5900 6550
@@
 $EndComp
 $Comp
-L GND #PWR17
+L GND #PWR016
 U 1 1 4FBE75E6
 P 6500 7350
-F 0 "#PWR17" H 6500 7350 30  0001 C CNN
+F 0 "#PWR016" H 6500 7350 30  0001 C CNN
 F 1 "GND" H 6500 7280 30  0001 C CNN
 	1    6500 7350
@@
 $EndComp
 $Comp
-L GND #PWR11
+L GND #PWR017
 U 1 1 4FB6D221
 P 5600 5550
-F 0 "#PWR11" H 5600 5550 30  0001 C CNN
+F 0 "#PWR017" H 5600 5550 30  0001 C CNN
 F 1 "GND" H 5600 5480 30  0001 C CNN
 	1    5600 5550
@@
 $EndComp
 $Comp
-L +3V #PWR10
+L +3V #PWR018
 U 1 1 4FB4FBCB
 P 5600 3950
-F 0 "#PWR10" H 5600 3860 30  0001 C CNN
+F 0 "#PWR018" H 5600 3860 30  0001 C CNN
 F 1 "+3V" H 5600 4060 30  0000 C CNN
 	1    5600 3950
@@
 $EndComp
 $Comp
-L GND #PWR18
+L GND #PWR019
 U 1 1 4FB4FBAE
 P 7500 7350
-F 0 "#PWR18" H 7500 7350 30  0001 C CNN
+F 0 "#PWR019" H 7500 7350 30  0001 C CNN
 F 1 "GND" H 7500 7280 30  0001 C CNN
 	1    7500 7350
@@
 WIFI_SLEEP
 $Comp
-L GND #PWR5
+L GND #PWR020
 U 1 1 4FB1371E
 P 3950 7600
-F 0 "#PWR5" H 3950 7600 30  0001 C CNN
+F 0 "#PWR020" H 3950 7600 30  0001 C CNN
 F 1 "GND" H 3950 7530 30  0001 C CNN
 	1    3950 7600
@@
 $EndComp
 $Comp
-L +3V #PWR1
+L +3V #PWR021
 U 1 1 4FB1357C
 P 850 3700
-F 0 "#PWR1" H 850 3610 30  0001 C CNN
+F 0 "#PWR021" H 850 3610 30  0001 C CNN
 F 1 "+3V" H 850 3810 30  0000 C CNN
 	1    850  3700
@@
 WIFI_TX
 $Comp
-L GND #PWR2
+L GND #PWR022
 U 1 1 4FB0BC87
 P 850 7350
-F 0 "#PWR2" H 850 7350 30  0001 C CNN
+F 0 "#PWR022" H 850 7350 30  0001 C CNN
 F 1 "GND" H 850 7280 30  0001 C CNN
 	1    850  7350
@@
 $EndComp
 $Comp
-L +3V #PWR25
+L +3V #PWR023
 U 1 1 4FB0AACD
 P 11500 850
-F 0 "#PWR25" H 11500 760 30  0001 C CNN
+F 0 "#PWR023" H 11500 760 30  0001 C CNN
 F 1 "+3V" H 11500 960 30  0000 C CNN
 	1    11500 850
@@
 $EndComp
 $Comp
-L +BATT #PWR26
+L +BATT #PWR024
 U 1 1 4FB0A598
 P 11800 850
-F 0 "#PWR26" H 11800 800 20  0001 C CNN
+F 0 "#PWR024" H 11800 800 20  0001 C CNN
 F 1 "+BATT" H 11800 950 30  0000 C CNN
 	1    11800 850
@@
 $EndComp
 $Comp
-L GND #PWR29
+L GND #PWR025
 U 1 1 4FB0A559
 P 12200 2450
-F 0 "#PWR29" H 12200 2450 30  0001 C CNN
+F 0 "#PWR025" H 12200 2450 30  0001 C CNN
 F 1 "GND" H 12200 2380 30  0001 C CNN
 	1    12200 2450
@@
 E-
 $Comp
-L GND #PWR28
+L GND #PWR026
 U 1 1 4FABACF9
 P 12150 7250
-F 0 "#PWR28" H 12150 7250 30  0001 C CNN
+F 0 "#PWR026" H 12150 7250 30  0001 C CNN
 F 1 "GND" H 12150 7180 30  0001 C CNN
 	1    12150 7250
@@
 $EndComp
 $Comp
-L PWR_FLAG #FLG1
+L PWR_FLAG #FLG027
 U 1 1 4F9C2D4F
 P 4100 1850
-F 0 "#FLG1" H 4100 2120 30  0001 C CNN
+F 0 "#FLG027" H 4100 2120 30  0001 C CNN
 F 1 "PWR_FLAG" H 4100 2080 30  0000 C CNN
 	1    4100 1850
@@
 D+
 $Comp
-L +VUSB #PWR4
+L +VUSB #PWR028
 U 1 1 4F9C233A
 P 2800 1450
-F 0 "#PWR4" H 2800 1400 20  0001 C CNN
+F 0 "#PWR028" H 2800 1400 20  0001 C CNN
 F 1 "+VUSB" H 2800 1550 30  0000 C CNN
 	1    2800 1450
@@
 $EndComp
 $Comp
-L +3V #PWR20
+L +3V #PWR029
 U 1 1 4F9C1A78
 P 8650 1450
-F 0 "#PWR20" H 8650 1360 30  0001 C CNN
+F 0 "#PWR029" H 8650 1360 30  0001 C CNN
 F 1 "+3V" H 8650 1560 30  0000 C CNN
 	1    8650 1450
@@
 $EndComp
 $Comp
-L +BATT #PWR6
+L +BATT #PWR030
 U 1 1 4F9C1A77
 P 5400 1450
-F 0 "#PWR6" H 5400 1400 20  0001 C CNN
+F 0 "#PWR030" H 5400 1400 20  0001 C CNN
 F 1 "+BATT" H 5400 1550 30  0000 C CNN
 	1    5400 1450
@@
 $EndComp
 $Comp
-L GND #PWR7
+L GND #PWR031
 U 1 1 4F9C1A76
 P 5400 2400
-F 0 "#PWR7" H 5400 2400 30  0001 C CNN
+F 0 "#PWR031" H 5400 2400 30  0001 C CNN
 F 1 "GND" H 5400 2330 30  0001 C CNN
 	1    5400 2400
@@
 MOSI
 $Comp
-L +3V #PWR23
+L +3V #PWR032
 U 1 1 4F9C1A71
 P 11400 9250
-F 0 "#PWR23" H 11400 9160 30  0001 C CNN
+F 0 "#PWR032" H 11400 9160 30  0001 C CNN
 F 1 "+3V" H 11400 9360 30  0000 C CNN
 	1    11400 9250
@@
 $EndComp
 $Comp
-L GND #PWR24
+L GND #PWR033
 U 1 1 4F9C1A70
 P 11400 10000
-F 0 "#PWR24" H 11400 10000 30  0001 C CNN
+F 0 "#PWR033" H 11400 10000 30  0001 C CNN
 F 1 "GND" H 11400 9930 30  0001 C CNN
 	1    11400 10000

Commit message: Add remaining test points
Parts:
- added P1, P10, P11, P18, P19, P2, P20, P21, P23, P24, P25, P26, P29, P32, P35, P38, P39, P40, P41, P42, P43, P6, P7, P8, P9: CONN_1, symbol CONN_1
- renumbered P4 to P12, P5 to P13, P6 to P14, P7 to P15, P8 to P16, P9 to P17, P10 to P22, P11 to P27, P12 to P28, P1 to P3, P13 to P30, P14 to P31, P15 to P33, P16 to P34, P17 to P36, P18 to P37, P2 to P4, P19 to P44, P3 to P5
Connections:
- net CHG: now also P18.1
- net I2C_CLOCK: now also P21.1
- net I2C_DATA: now also P19.1
- net LCD_CLOCK: now also P20.1
- net WIFI_ASSOC: now also P11.1
- net WIFI_CTS: now also P7.1
- net WIFI_RESET: now also P1.1
- net WIFI_RTS: now also P6.1
- net WIFI_RX: now also P8.1
- net WIFI_SLEEP: now also P10.1
- net WIFI_TX: now also P9.1
- net WIFI_WAKE: now also P2.1
- net at P44.1 (P1), U5.13 (BP0): now also P23.1
- net at P44.10 (P10), U5.22 (S5): now also P40.1
- net at P44.11 (P11), U5.23 (S6): now also P41.1
- net at P44.12 (P12), U5.24 (S7): now also P42.1
- net at P44.13 (P13), U5.25 (S8): now also P43.1
- net at P44.2 (P2), U5.14 (BP1): now also P24.1
- net at P44.3 (P3), U5.15 (BP2): now also P25.1
- net at P44.4 (P4), U5.16 (BP3): now also P26.1
- net at P44.5 (P5), U5.17 (S0): now also P29.1
- net at P44.6 (P6), U5.18 (S1): now also P32.1
- net at P44.7 (P7), U5.19 (S2): now also P35.1
- net at P44.8 (P8), U5.20 (S3): now also P38.1
- net at P44.9 (P9), U5.21 (S4): now also P39.1
Other:
- moved on the sheet: D1, R12, R13, R14
