File: hardware/WeighFi.sch (KiCad schematic (older format))
At the start: 101 parts, among them P1 CONN_1, P10 CONN_1, P11 CONN_1, P12 CONN_1, P13 CONN_1, P14 CONN_1, P15 CONN_1, P16 CONN_1, P17 CONN_1, P18 CONN_1, P19 CONN_1, P2 CONN_1, P20 CONN_1, P21 CONN_1, P22 CONN_4, P23 CONN_1, P24 CONN_1, P25 CONN_1, P26 CONN_1, P27 CONN_1, P28 CONN_1, P29 CONN_1, P3 CONN_1, P30 CONN_1, P31 CONN_1, P32 CONN_1, P33 CONN_1, P34 CONN_1, P35 CONN_1, P36 CONN_1, P37 CONN_1, P38 CONN_1, P39 CONN_1, P4 CONN_1, P40 CONN_1, P41 CONN_1, P42 CONN_1, P43 CONN_1, P44 CONN_13, P5 CONN_1, P6 CONN_1, P7 CONN_1, P8 CONN_1, P9 CONN_1, Q1 MOSFET_P, U1 MAX1555, U2 MCP1700, U3 ATMEGA16U4/32U4, U4 ADS1131, U5 PCF8566, X1 CRYSTAL

Commit message: Move combined power & display units switch to individual switches. Add a status LED.
Parts:
- removed S1: SWITCH_DP4T, symbol SWITCH_DP4T
- added D2: LED, symbol LED
- added P19: CONN_1, symbol CONN_1
- added R13: 1K8, symbol R
- added S2: SWITCH_SPDT, symbol SWITCH_SPDT
- added S3: SWITCH_SP3T, symbol SWITCH_SP3T
- renumbered H5 to H2, H2 to H3, H6 to H4, H3 to H5, H7 to H6, H4 to H7, P19 to P20, P20 to P21, P21 to P22, P22 to P23, P23 to P24, P24 to P25, P25 to P26, P26 to P27, P29 to P28, P27 to P29, P28 to P30, P32 to P31, P30 to P32, P31 to P33, P35 to P34, P33 to P35, P34 to P36, P38 to P37, P36 to P38, P37 to P39, P39 to P40, P40 to P41, P41 to P42, P42 to P43, P43 to P44, P44 to P45, R13 to R14, R14 to R15, S2 to S1
Connections:
- net +BATT: now also S2.2
- net GND: now also D2.2 (K), S3.2
- net PWR_SW_OUT: now also S2.3
- net SW_KG: now also S3.1
- net SW_LB: now also S3.3
- net SW_ST: now also S3.4
- net STATUS: now reaches U3.40 ((ADC1)_PF1)
- net STATUS: now also P19.1, R13.1
- new net: D2.1 (A), R13.2
- no-connect marks 38 -> 36
Other:
- note added: "In System Programming header"
- note added: "Power, unit selection, and bootloader switches"
- note added: "Status LEDs"
- note removed: "Charging status display"
- note removed: "In System Programming header\nand reset to bootloader switch"
- note removed: "Main power and unit selection switch"
- moved on the sheet: D1, P18, P3, P4, P5, R12, S1

Commit message: More footprint assignments, add debug jumper
Parts:
- removed S1: SWITCH_SPST, symbol SWITCH_SPST
- added JP1: JUMPER, symbol JUMPER
- added S3: SWITCH_PUSH_NO, symbol SWITCH_PUSH_NO
- renumbered S2 to S1, S3 to S2
Connections:
- net GND: now also JP1.2, S3.2
- net RST: now also S3.1
- net DEBUG: now reaches U3.1 ((INT.6/AIN0)_PE6)
- net DEBUG: now also JP1.1
- no-connect marks 36 -> 35
Other:
- note added: "In System Programming header\nand reset pushbutton"
- note added: "Power and display unit switches,\ndebug mode jumper"
- note removed: "In System Programming header"
- note removed: "Power, unit selection, and bootloader switches"
- moved on the sheet: P3, P4, P5, S1, S2

Commit message: More footprint assignments, revisit board outline and enclosure features
Connections:
- net +BATT: now also P23.2; no longer P23.3
- net E-: now also P23.1; no longer P23.4
- net S+: now also P23.4; no longer P23.1
- net S-: now also P23.3; no longer P23.2
Other:
- note added: "Main power switch, display units switch,\ndebug mode jumper"
- note removed: "Power and display unit switches,\ndebug mode jumper"
Changed lines of the file:
@@
-EESchema Schematic File Version 2  date Tue 26 Jun 2012 19:12:08 BST
+EESchema Schematic File Version 2  date Wed 27 Jun 2012 17:24:55 BST
 LIBS:dresco
 LIBS:WeighFi-cache
@@
 Sheet 1 1
 Title "WeighFi"
-Date "26 jun 2012"
+Date "27 jun 2012"
 Rev "1.0"
 Comp ""
@@
 	1    0    0    -1
 $EndComp
+Text GLabel 12600 9500 0    60   Input ~ 0
+E-
+Text GLabel 12600 9600 0    60   Input ~ 0
+E+
+Text GLabel 12600 9700 0    60   Input ~ 0
+S-
 Text GLabel 12600 9800 0    60   Input ~ 0
-E-
-Text GLabel 12600 9700 0    60   Input ~ 0
-E+
-Text GLabel 12600 9600 0    60   Input ~ 0
-S-
-Text GLabel 12600 9500 0    60   Input ~ 0
 S+
 $Comp
@@
 Strain gauge connector
 Text Notes 700  8900 0    60   ~ 0
-Power and display unit switches,\ndebug mode jumper
+Main power switch, display units switch,\ndebug mode jumper
 Text Notes 4400 8900 0    60   ~ 0
 Voltage divider for \nbattery measurements \nusing internal ADC
