File: hardware/WeighFi-Main.sch (KiCad schematic (older format))
At the start: 69 parts, among them P1 CONN_1, P10 CONN_1, P11 CONN_1, P12 CONN_1, P13 CONN_1, P14 CONN_1, P15 CONN_1, P16 CONN_1, P17 CONN_1, P18 CONN_1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

Commit message: Refine schematics, generate new netlists
Parts:
- renumbered C9 to C10, C10 to C11, C11 to C12, C12 to C9, R9 to R10, R10 to R8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
Other:
- moved on the sheet: ANT1, C10, C11, C12, C13, C14, C5, C6, C7, C8, D1, D2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
