File: hardware/Main/WeighFi-Main.sch (KiCad schematic (older format))
At the start: 69 parts, among them P1 CONN_1, P10 CONN_1, P11 CONN_1, P12 CONN_1, P13 CONN_1, P14 CONN_1, P15 CONN_1, P16 CONN_1, P17 CONN_1, P18 CONN_1, P19 CONN_1, P2 CONN_1, P20 CONN_12, P3 CONN_1, P4 CONN_1, P5 CONN_1, P6 CONN_1, P7 CONN_1, P8 CONN_1, P9 CONN_1, Q1 MOSFET_P, U1 MAX1555, U2 MCP1700, U3 ATMEGA16U4/32U4, X1 CRYSTAL

Commit message: Replace RN-171 wireless module with ESP-03
Parts:
- removed ANT1: ANTENNA, symbol ANTENNA
- removed MOD1: RN-171, symbol RN-171
- removed P10, P11, P6, P8: CONN_1, symbol CONN_1
- removed R1, R2, R3, R4: R, symbol R
- added MOD1: ESP8266-ESP-03, symbol ESP8266-ESP-03
- renumbered P14 to P10, P15 to P11, P16 to P12, P17 to P13, P18 to P14, P19 to P15, P20 to P16, P9 to P3, P3 to P4, P4 to P5, P5 to P6, P12 to P8, P13 to P9, R5 to R1, R6 to R2, R7 to R3, R8 to R4, R9 to R5, R10 to R6, R11 to R7, R12 to R8, R13 to R9
Connections:
- net +3V: now also MOD1.8 (VCC)
- net GND: now also MOD1.1 (GND), MOD1.12 (GPIO15)
- net WIFI_RESET: now also MOD1.6 (CH_PD)
- net WIFI_RX: now also P3.1, MOD1.4 (RX)
- net WIFI_TX: now also P2.1, MOD1.3 (TX); no longer P3.1
- net WIFI_ASSOC renamed WIFI_BOOTLDR
- net WIFI_BOOTLDR: now also P7.1, MOD1.14 (GPIO0)
- net WIFI_CTS: no longer names the net of U3.12 ((PCINT7/OC0A/OC1C/RTS)_PB7)
- net WIFI_CTS: no longer P7.1
- net WIFI_RTS: no longer names the net of U3.22 ((XCK1/CTS)_PD5)
- net WIFI_SLEEP: no longer names the net of U3.37 ((TDO/ADC6)_PF6)
- net WIFI_WAKE: no longer names the net of U3.36 ((TDI/ADC7)_PF7)
- net WIFI_WAKE: no longer P2.1
- no-connect marks 20 -> 14
Other:
- note removed: "Optional circuitry to support\nwake on CTS or received data"
- note removed: "The RTS and CTS signals are unlikely to be used,\ncould be dropped if routing is problematic."
- moved on the sheet: P1, P2, P3

Commit message: Shuffle some MCU pin connections and labels, add a vibration switch as additional wake up source.
Parts:
- added P17: CONN_1, symbol CONN_1
- added R10: 1M, ~, symbol R
- added S4: SWITCH_VIBRATION, symbol SWITCH_VIBRATION
Connections:
- net +3V: now also R10.2
- net ADC_SPEED: now also U3.25 ((PCINT20/XCK/T0)_PD4); no longer U3.31 ((OC3A/OC4A)_PC6)
- net GND: now also S4.1
- net LCD_CLOCK: now also U3.32 ((ICP3/CLK0/OC4A)_PC7); no longer U3.29 ((PCINT5/OC1A/OC4B/ADC12)_PB5)
- net LCD_ENABLE: now also U3.31 ((OC3A/OC4A)_PC6); no longer U3.25 ((PCINT20/XCK/T0)_PD4)
- net STATUS: now also U3.36 ((TDI/ADC7)_PF7); no longer U3.40 ((ADC1)_PF1)
- net SW_ST: now also U3.29 ((PCINT5/OC1A/OC4B/ADC12)_PB5); no longer U3.8 ((PCINT0/SS)_PB0)
- net WIFI_BOOTLDR: now also U3.37 ((TDO/ADC6)_PF6); no longer U3.38 ((TMS/ADC5)_PF5)
- net MCU_WAKE: now reaches U3.12 ((PCINT7/OC0A/OC1C/RTS)_PB7)
- net MCU_WAKE: now also P17.1, R10.1, S4.2
- net ADC_ENABLE: now reaches U3.22 ((XCK1/CTS)_PD5)
- net ADC_ENABLE: now also P16.6 (P6)
- removed net ADC_PWRDN: P16.6 (P6), U3.32 ((ICP3/CLK0/OC4A)_PC7)
- net WIFI_RESET renamed WIFI_ENABLE
- net WIFI_ENABLE: now also U3.38 ((TMS/ADC5)_PF5); no longer U3.39 ((TCK/ADC4)_PF4)
- no-connect marks 14 -> 13
Other:
- note added: "Vibration Sensor"

Commit message: Update power supply for 3xAA alkaline batteries
Still using an LDO for low noise and low quiescent current.
May migrate to switcher for increased efficiency in a future
revision (noting that ADC reference comes direct from battery,
which should lower the impact of any switching noise).

Remove USB LiPo charging circuitry.

Add large capacitor to give the batteries an easier time with
current peaks from WiFi transmission.
Parts:
- removed C1, C2: 1uF, symbol C
- removed D1: LED, symbol LED
- removed P14: CONN_1, symbol CONN_1
- removed R8: 1K8, symbol R
- removed U1: MAX1555, symbol MAX1555
- C1: renamed from C3; value 1uF -> 330uF
- renumbered C11 to C10, C12 to C11, C13 to C12, C14 to C13, C9 to C2, C15 to C3, C10 to C9, D2 to D1, P9 to P1, P12 to P10, P8 to P11, P15 to P12, P11 to P13, P13 to P14, P17 to P15, P10 to P2, P1 to P3, P2 to P4, P3 to P5, P4 to P6, P5 to P7, P6 to P8, P7 to P9, R9 to R4, R4 to R5, R5 to R6, R6 to R7, R7 to R8, R10 to R9, U2 to U1, U3 to U2
Other:
- note added: "Power supply"
- note added: "Status LED"
- note added: "USB connector"
- note removed: "Status LEDs"
- note removed: "USB, LiPo charging, and power supply"
- moved on the sheet: BT1, C1, C2, C3, D1, P1, P10, P12, P2, R4, U1, USB1

Commit message: Current limiting resistors between MCU and WiFi module
Some protection for the microcontroller, just in case. Have
seen one instance of a faulty/damaged ESP8266 module pulling
excess current from the CH_PD pin.
Parts:
- removed C1: 330uF, symbol C
- added C1: 330uF, ~, symbol CP
- added R10, R11, R12, R9: 100, symbol R
- renumbered R9 to R13, R6 to R4, R7 to R5, R4 to R6, R5 to R7
Connections:
- wire segments 174 -> 178
Other:
- moved on the sheet: C10, C11, C12, C13, C5, C6, C7, C8, C9, L1, R3, R4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

Commit message: Pin swaps to aid board routing
Parts:
- R1: value R -> 670K
- R2: value R -> 470K
- renumbered R12 to R10, R10 to R11, R9 to R12, R11 to R9
Other:
- moved on the sheet: R11, R12
Changed lines of the file:
@@
 Text GLabel 7200 1100 0    60   Input ~ 0
 STATUS
-Text GLabel 10350 4750 2    60   Input ~ 0
+Text GLabel 10350 6450 2    60   Input ~ 0
 STATUS
 $Comp
@@
 Text Notes 7000 700  0    60   ~ 0
 Status LED
-Text GLabel 11350 4550 2    60   Input ~ 0
+Text GLabel 11350 5750 2    60   Input ~ 0
 WIFI_ENABLE
-Text GLabel 10350 6250 2    60   Input ~ 0
+Text GLabel 10350 7050 2    60   Input ~ 0
 LCD_CLOCK
 $Comp
@@
 Text GLabel 1900 4950 0    60   Input ~ 0
 WIFI_ENABLE
-Text GLabel 10350 7050 2    60   Input ~ 0
+Text GLabel 10350 4750 2    60   Input ~ 0
 SW_KG
-Text GLabel 10350 6850 2    60   Input ~ 0
+Text GLabel 10350 4650 2    60   Input ~ 0
 SW_LB
-Text GLabel 10350 6950 2    60   Input ~ 0
+Text GLabel 10350 4550 2    60   Input ~ 0
 SW_ST
 Text GLabel 3100 10200 2    60   Input ~ 0
@@
 PWR_SW_OUT
 NoConn ~ 2600 9250
-Text GLabel 10350 5750 2    60   Input ~ 0
+Text GLabel 10350 6850 2    60   Input ~ 0
 ADC_ENABLE
-Text GLabel 10350 5650 2    60   Input ~ 0
+Text GLabel 10350 6950 2    60   Input ~ 0
 ADC_SPEED
+Text GLabel 10350 5850 2    60   Input ~ 0
+ADC_DATA
 Text GLabel 10350 5950 2    60   Input ~ 0
-ADC_DATA
-Text GLabel 10350 5850 2    60   Input ~ 0
 ADC_CLOCK
 $Comp
@@
 P 5550 9950
 F 0 "R2" V 5630 9950 50  0000 C CNN
-F 1 "R" V 5550 9950 50  0000 C CNN
+F 1 "470K" V 5550 9950 50  0000 C CNN
 F 2 "" H 5550 9950 60  0001 C CNN
 F 3 "" H 5550 9950 60  0001 C CNN
@@
 P 5550 9250
 F 0 "R1" V 5630 9250 50  0000 C CNN
-F 1 "R" V 5550 9250 50  0000 C CNN
+F 1 "670K" V 5550 9250 50  0000 C CNN
 F 2 "" H 5550 9250 60  0001 C CNN
 F 3 "" H 5550 9250 60  0001 C CNN
@@
 $EndComp
 NoConn ~ 2450 5300
-Text GLabel 11350 4650 2    60   Input ~ 0
+Text GLabel 11350 5650 2    60   Input ~ 0
 WIFI_BOOTLDR
 $Comp
@@
 NoConn ~ 10050 4350
 NoConn ~ 10050 4450
-NoConn ~ 10050 6450
 $Comp
 L R R13
@@
 	13250 2150 13250 2250
 Wire Wire Line
-	10050 4950 10350 4950
-Wire Wire Line
 	1800 10750 1400 10750
 Connection ~ 11500 10200
@@
 	15750 8450 750  8450
 Wire Wire Line
-	10050 6850 10350 6850
-Wire Wire Line
 	2600 10200 3100 10200
 Wire Wire Line
@@
 Wire Wire Line
 	2600 9450 3100 9450
-Wire Wire Line
-	10050 5950 10350 5950
 Connection ~ 5550 10300
 Wire Wire Line
@@
 Connection ~ 5200 9600
 Wire Wire Line
-	10050 5850 10350 5850
-Wire Wire Line
 	1400 9350 1650 9350
 Wire Wire Line
@@
 Wire Wire Line
 	2600 10100 3100 10100
-Wire Wire Line
-	10050 7050 10350 7050
 Wire Notes Line
 	15750 3050 750  3050
@@
 	3800 4250 3800 4700
 Connection ~ 3800 4700
-Wire Wire Line
-	10350 6950 10050 6950
-Wire Wire Line
-	10350 4750 10050 4750
-Wire Wire Line
-	10050 5650 10350 5650
-Wire Wire Line
-	10350 5750 10050 5750
-Wire Wire Line
-	10050 6150 10350 6150
-Wire Wire Line
-	10350 6250 10050 6250
-Wire Wire Line
-	10050 7150 10350 7150
 Wire Wire Line
 	13650 4250 13650 4400
@@
 $EndComp
 $Comp
+L R R12
+U 1 1 554FA8A3
+P 11000 5750
+F 0 "R12" V 11050 5550 50  0000 C CNN
+F 1 "100" V 11000 5750 50  0000 C CNN
+F 2 "" H 11000 5750 60  0001 C CNN
+F 3 "" H 11000 5750 60  0001 C CNN
+	1    11000 5750
+	0    -1   -1   0
+$EndComp
+$Comp
+L R R11
+U 1 1 554FA8F4
+P 11000 5650
+F 0 "R11" V 11050 5450 50  0000 C CNN
+F 1 "100" V 11000 5650 50  0000 C CNN
+F 2 "" H 11000 5650 60  0001 C CNN
+F 3 "" H 11000 5650 60  0001 C CNN
+	1    11000 5650
+	0    -1   -1   0
+$EndComp
+$Comp
 L R R9
-U 1 1 554FA8A3
-P 11000 4550
-F 0 "R9" V 11050 4350 50  0000 C CNN
-F 1 "100" V 11000 4550 50  0000 C CNN
-F 2 "" H 11000 4550 60  0001 C CNN
-F 3 "" H 11000 4550 60  0001 C CNN
-	1    11000 4550
-	0    -1   -1   0
-$EndComp
-$Comp
-L R R10
-U 1 1 554FA8F4
-P 11000 4650
-F 0 "R10" V 11050 4450 50  0000 C CNN
-F 1 "100" V 11000 4650 50  0000 C CNN
-F 2 "" H 11000 4650 60  0001 C CNN
-F 3 "" H 11000 4650 60  0001 C CNN
-	1    11000 4650
-	0    -1   -1   0
-$EndComp
-$Comp
-L R R11
 U 1 1 554FA8FF
 P 11000 5450
-F 0 "R11" V 11050 5250 50  0000 C CNN
+F 0 "R9" V 11050 5250 50  0000 C CNN
 F 1 "100" V 11000 5450 50  0000 C CNN
 F 2 "" H 11000 5450 60  0001 C CNN
@@
 $EndComp
 $Comp
-L R R12
+L R R10
 U 1 1 554FA90A
 P 11000 5550
-F 0 "R12" V 11050 5350 50  0000 C CNN
+F 0 "R10" V 11050 5350 50  0000 C CNN
 F 1 "100" V 11000 5550 50  0000 C CNN
 F 2 "" H 11000 5550 60  0001 C CNN
@@
 $EndComp
 Wire Wire Line
-	10050 4550 10750 4550
-Wire Wire Line
-	10050 4650 10750 4650
-Wire Wire Line
-	11250 4550 11350 4550
-Wire Wire Line
-	11250 4650 11350 4650
+	11250 5750 11350 5750
+Wire Wire Line
+	11250 5650 11350 5650
 Wire Wire Line
 	10050 5450 10750 5450
@@
 Wire Wire Line
 	11250 5550 11350 5550
+Wire Wire Line
+	10350 4550 10050 4550
+Wire Wire Line
+	10350 4650 10050 4650
+Wire Wire Line
+	10350 4750 10050 4750
+Wire Wire Line
+	10750 5650 10050 5650
+Wire Wire Line
+	10750 5750 10050 5750
+Wire Wire Line
+	10350 5850 10050 5850
+Wire Wire Line
+	10350 5950 10050 5950
+Wire Wire Line
+	10350 6150 10050 6150
+Wire Wire Line
+	10350 6850 10050 6850
+Wire Wire Line
+	10350 6950 10050 6950
+Wire Wire Line
+	10350 7050 10050 7050
+Wire Wire Line
+	10350 7150 10050 7150
+Wire Wire Line
+	10350 6450 10050 6450
+NoConn ~ 10050 6250
+Wire Wire Line
+	10350 4950 10050 4950
 $EndSCHEMATC

Commit message: Add additional capacitor on 3v rail
Parts:
- added C14: 330uF, ~, symbol CP
Connections:
- wire segments 178 -> 180
Other:
- moved on the sheet: P10
Changed lines of the file:
@@
 L +3V #PWR025
 U 1 1 4F9C1A78
-P 4950 1450
-F 0 "#PWR025" H 4950 1360 30  0001 C CNN
-F 1 "+3V" H 4950 1560 30  0000 C CNN
-F 2 "" H 4950 1450 60  0001 C CNN
-F 3 "" H 4950 1450 60  0001 C CNN
-	1    4950 1450
+P 5350 1450
+F 0 "#PWR025" H 5350 1360 30  0001 C CNN
+F 1 "+3V" H 5350 1560 30  0000 C CNN
+F 2 "" H 5350 1450 60  0001 C CNN
+F 3 "" H 5350 1450 60  0001 C CNN
+	1    5350 1450
 	1    0    0    -1
 $EndComp
@@
 L CONN_1 P10
 U 1 1 4F9C1A69
-P 4750 1450
-F 0 "P10" H 4830 1450 40  0000 L CNN
-F 1 "CONN_1" H 4750 1505 30  0001 C CNN
-F 2 "" H 4750 1450 60  0001 C CNN
-F 3 "" H 4750 1450 60  0001 C CNN
-	1    4750 1450
+P 5200 1450
+F 0 "P10" H 5280 1450 40  0000 L CNN
+F 1 "CONN_1" H 5200 1505 30  0001 C CNN
+F 2 "" H 5200 1450 60  0001 C CNN
+F 3 "" H 5200 1450 60  0001 C CNN
+	1    5200 1450
 	0    -1   -1   0
 $EndComp
@@
 	3950 2200 3950 1900
 Wire Wire Line
-	4950 1600 4950 1450
+	5350 1600 5350 1450
 Wire Wire Line
 	1700 2200 1700 2400
@@
 Wire Wire Line
 	11500 9700 11250 9700
-Connection ~ 4750 1600
+Connection ~ 5200 1600
 Connection ~ 1900 1600
 Connection ~ 1900 2200
@@
 	4100 8700 4100 11000
 Wire Wire Line
-	4350 1600 4950 1600
+	4350 1600 5350 1600
 Wire Wire Line
 	3450 2200 3450 2300
@@
 USB connector
 Wire Wire Line
-	950  2200 4550 2200
+	950  2200 4950 2200
 Wire Wire Line
 	1450 1700 1450 1600
@@
 Wire Wire Line
 	10350 4950 10050 4950
+$Comp
+L CP C14
+U 1 1 55608D98
+P 4950 1950
+F 0 "C14" H 5000 2050 50  0000 L CNN
+F 1 "330uF" H 5000 1830 50  0000 L CNN
+F 2 "~" H 4950 1950 60  0000 C CNN
+F 3 "~" H 4950 1950 60  0000 C CNN
+	1    4950 1950
+	1    0    0    -1
+$EndComp
+Wire Wire Line
+	4950 1750 4950 1600
+Connection ~ 4950 1600
+Wire Wire Line
+	4950 2200 4950 2150
+Connection ~ 4550 2200
 $EndSCHEMATC
