File: hardware/Main/WeighFi-Main.sch (KiCad schematic (older format))
At the start: 62 parts, among them P1 CONN_1, P10 CONN_1, P11 CONN_1, P12 CONN_1, P13 CONN_1, P14 CONN_1, P15 CONN_1, P16 CONN_12, P2 CONN_1, P3 CONN_1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

Commit message: Voltage divider resistors swapped in schematic and netlist
Parts:
- R1: value 670K -> 470K
- R2: value 470K -> 680K
Changed lines of the file:
@@
 P 5550 9950
 F 0 "R2" V 5630 9950 50  0000 C CNN
-F 1 "470K" V 5550 9950 50  0000 C CNN
+F 1 "680K" V 5550 9950 50  0000 C CNN
 F 2 "" H 5550 9950 60  0001 C CNN
 F 3 "" H 5550 9950 60  0001 C CNN
@@
 P 5550 9250
 F 0 "R1" V 5630 9250 50  0000 C CNN
-F 1 "670K" V 5550 9250 50  0000 C CNN
+F 1 "470K" V 5550 9250 50  0000 C CNN
 F 2 "" H 5550 9250 60  0001 C CNN
 F 3 "" H 5550 9250 60  0001 C CNN
